File: Senior_Design_PCB_ethanl7_nrkim2/Senior_Design_PCB_ethanl7_nrkim2.kicad_sch (KiCad schematic)
At the start: 83 parts, among them J1 Piezo, J10 M6, J2 9V supply battery or bench, J3 Conn_02x03_Odd_Even, J4 Conn_ARM_JTAG_SWD_10, J5 M1, J6 M2, J7 M3, J8 M4, J9 M5, SW1 SW_Push, U1 uA7805, U2 LM386, U3 L298N, U4 L298N, U5 L298N, U6 STM32H7B0RBTx, U7 LM2937xT

Commit message: finished v1 pcb design
Parts:
- added C19: 100 nF, Capacitor_SMD:C_0805_2012Metric_Pad1.18x1.45mm_HandSolder, symbol Device:C
- added R11: 10 kOhm, Resistor_SMD:R_0805_2012Metric_Pad1.20x1.40mm_HandSolder, symbol Device:R
- added R12: 20 kOhm, Resistor_SMD:R_0805_2012Metric_Pad1.20x1.40mm_HandSolder, symbol Device:R
- D1, D2: footprint LED_SMD:LED_0805_2012Metric_Pad1.15x1.40mm_HandSolder -> Connector_Molex:Molex_KK-254_AE-6410-02A_1x02_P2.54mm_Vertical
Connections:
- net +5V: now also C19.2; no longer U2.6 (V+)
- net Amp_Sig: now also R11.2, R12.2; no longer TP2.1, U2.5
- net GND: now also R12.1
- net M1N: now also U6.36 (PB15); no longer U6.28 (PB2)
- net M1P: now also U6.35 (PB14); no longer U6.27 (PB1)
- net M2N: now also U6.38 (PC7); no longer U6.33 (PB12)
- net M2P: now also U6.37 (PC6); no longer U6.29 (PB10)
- net M3N: now also U6.42 (PA10); no longer U6.36 (PB15)
- net M3P: now also U6.41 (PA9); no longer U6.35 (PB14)
- net M4N: now also U6.52 (PC11); no longer U6.38 (PC7)
- net M4P: now also U6.51 (PC10); no longer U6.37 (PC6)
- net M5N: now also U6.28 (PB2); no longer U6.42 (PA10)
- net M5P: now also U6.27 (PB1); no longer U6.41 (PA9)
- net M6N: now also U6.33 (PB12); no longer U6.52 (PC11)
- net M6P: now also U6.29 (PB10); no longer U6.51 (PC10)
- net at D1.2 (A): now also U6.58 (PB6); no longer U6.57 (PB5)
- net at D2.2 (A): now also U6.57 (PB5); no longer U6.58 (PB6)
- new net: R11.1, TP2.1, U2.5
- new net: C19.1, U2.6 (V+)
- no-connect marks 30 -> 29
Other:
- note removed: "might need volt divider"
- moved on the sheet: TP2
